File: BlinkenHeart.kicad_pcb (KiCad board)
At the start: 2 copper layers, 84.7 x 74 mm, 28 parts, among them IC1 ATTINY85-S, SW1 Taster, SW2 Schalter

Commit message: Did some rerouting
Parts:
- turned D11 to 153 degrees
- turned D12 to 180 degrees
- turned D2 to 145.5 degrees
- turned D3 to 90 degrees
- turned D6 to 0 degrees
- turned D9 to 270 degrees
Routing:
- net Net-(D10-Pad1): track 36.9 -> 45.2 mm, vias 0 -> 2
- net Net-(D7-Pad1): track 84.3 -> 92.5 mm, vias 4 -> 6
- net Net-(IC1-Pad3): track 66.7 -> 60.0 mm
- net Net-(D4-Pad1): track 100.9 -> 105.2 mm, vias 2 -> 4
- net 3: track 128.2 -> 125.4 mm, vias 7 -> 5
- net 1: track 142.6 -> 140.2 mm, vias 12 -> 7
- net Net-(D1-Pad1): track 85.4 -> 83.1 mm, vias 0 -> 4
- net 2: track 129.6 -> 131.0 mm, vias 8 -> 9
- net 4: track 171.1 -> 170.7 mm, vias 8 -> 6
- net RST: vias 3 -> 1

Commit message: Some rerouting (by Carsten)
Parts:
- moved IC1 201.3 mm to (49.5, 112.0)
- moved ? 201.1 mm to (95.6, 99.0)
- moved ? 201.1 mm to (55.0, 99.0)
- moved D13 201.1 mm to (62.9, 137.1)
- moved G*** 201.1 mm to (81.7, 151.8)
- moved BT1 201.1 mm to (58.7, 126.8)
- moved D1 201.1 mm to (86.7, 100.8)
- moved D10 201.1 mm to (45.7, 101.8)
- moved D11 201.1 mm to (64.7, 100.8)
- moved D12 201.1 mm to (75.7, 110.8)
- moved D2 201.1 mm to (105.7, 101.8)
- moved D3 201.1 mm to (114.7, 116.8)
- moved D4 201.1 mm to (106.7, 131.8)
- moved D5 201.1 mm to (90.7, 147.8)
- moved D6 201.1 mm to (75.7, 162.8)
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Routing:
- net GND: track 142.5 -> 106.1 mm, vias 4 -> 1
- net 4: track 170.7 -> 152.1 mm, vias 6 -> 5
- net Net-(D7-Pad1): track 92.5 -> 75.4 mm, vias 6 -> 4
- net VCC: track 76.1 -> 88.2 mm
- net Net-(D13-Pad1): track 9.67 -> 20.1 mm
- net 1: track 140.2 -> 130.3 mm, vias 7 -> 3
- net Net-(D4-Pad1): track 105.2 -> 98.5 mm, vias 4 -> 2
- net Net-(D10-Pad1): track 45.2 -> 39.8 mm, vias 2 -> 0
- net Net-(D1-Pad1): track 83.1 -> 87.8 mm, vias 4 -> 0
- net 2: track 131.0 -> 126.4 mm, vias 9 -> 5
- net 3: track 125.4 -> 123.4 mm, vias 5 -> 6
- net RST: track 65.8 -> 64.8 mm, vias 1 -> 2
- net Net-(IC1-Pad3): track 60.0 -> 59.5 mm, vias 4 -> 0
