File: BlinkenHeart.kicad_pcb (KiCad board)
At the start: 2 copper layers, 84.7 x 74 mm, 28 parts, among them IC1 ATTINY85-S, SW1 Taster, SW2 Schalter

Commit message: Final rotation
Parts:
- moved SW2 0.70 mm to (75.8, 143.2)
Other:
- board text added: "aus"
Changed lines of the file:
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@@
     (area 33.267868 94.910319 118.138681 169.044001)
     (thickness 1.6)
-    (drawings 10)
+    (drawings 11)
     (tracks 296)
     (zones 0)
@@
     (pad_to_mask_clearance 0.2)
     (aux_axis_origin 137 81)
-    (visible_elements 7FFFFFFF)
+    (visible_elements 7FFFFF7F)
     (pcbplotparams
       (layerselection 0x0103c_80000001)
@@
     (tags "LED led 1206 SMD smd SMT smt smdled SMDLED smtled SMTLED")
     (attr smd)
-    (fp_text reference D9 (at 0 2 270) (layer F.SilkS)
-      (effects (font (size 1 1) (thickness 0.15)))
-    )
-    (fp_text value LED (at 0 -2 270) (layer F.SilkS)
+    (fp_text reference D9 (at -0.146 -1.797 270) (layer F.SilkS)
+      (effects (font (size 1 1) (thickness 0.15)))
+    )
+    (fp_text value LED (at -0.046 1.753 450) (layer F.SilkS)
       (effects (font (size 1 1) (thickness 0.15)))
     )
@@
     (tags "LED led 1206 SMD smd SMT smt smdled SMDLED smtled SMTLED")
     (attr smd)
-    (fp_text reference D12 (at 0 2 180) (layer F.SilkS)
-      (effects (font (size 1 1) (thickness 0.15)))
-    )
-    (fp_text value LED (at 0 -2 180) (layer F.SilkS)
+    (fp_text reference D12 (at 0.078 -1.779 180) (layer F.SilkS)
+      (effects (font (size 1 1) (thickness 0.15)))
+    )
+    (fp_text value LED (at -0.022 1.746 180) (layer F.SilkS)
       (effects (font (size 1 1) (thickness 0.15)))
     )
@@
     (tags "LED led 1206 SMD smd SMT smt smdled SMDLED smtled SMTLED")
     (attr smd)
-    (fp_text reference D1 (at -0.07201 1.866451 212) (layer F.SilkS)
-      (effects (font (size 1 1) (thickness 0.15)))
-    )
-    (fp_text value LED (at -0.067048 -1.726942 212) (layer F.SilkS)
+    (fp_text reference D1 (at 0.057501 -1.737554 212) (layer F.SilkS)
+      (effects (font (size 1 1) (thickness 0.15)))
+    )
+    (fp_text value LED (at -0.050809 1.879699 212) (layer F.SilkS)
       (effects (font (size 1 1) (thickness 0.15)))
     )
@@
     (tags "LED led 1206 SMD smd SMT smt smdled SMDLED smtled SMTLED")
     (attr smd)
-    (fp_text reference D2 (at 0.308686 2.214659 145.5) (layer F.SilkS)
-      (effects (font (size 1 1) (thickness 0.15)))
-    )
-    (fp_text value LED (at 0.009765 -1.938454 145.5) (layer F.SilkS)
+    (fp_text reference D2 (at 0.085457 -1.823026 145.5) (layer F.SilkS)
+      (effects (font (size 1 1) (thickness 0.15)))
+    )
+    (fp_text value LED (at 0.012804 1.867126 145.5) (layer F.SilkS)
       (effects (font (size 1 1) (thickness 0.15)))
     )
@@
     (tags "LED led 1206 SMD smd SMT smt smdled SMDLED smtled SMTLED")
     (attr smd)
-    (fp_text reference D11 (at 0.016974 2.236004 153) (layer F.SilkS)
-      (effects (font (size 1 1) (thickness 0.15)))
-    )
-    (fp_text value LED (at 0.123568 -1.867661 153) (layer F.SilkS)
+    (fp_text reference D11 (at 0.031403 -1.872328 153) (layer F.SilkS)
+      (effects (font (size 1 1) (thickness 0.15)))
+    )
+    (fp_text value LED (at -0.01834 1.884752 153) (layer F.SilkS)
       (effects (font (size 1 1) (thickness 0.15)))
     )
@@
     (tags "LED led 1206 SMD smd SMT smt smdled SMDLED smtled SMTLED")
     (attr smd)
-    (fp_text reference D10 (at 0.075967 1.857324 208.5) (layer F.SilkS)
-      (effects (font (size 1 1) (thickness 0.15)))
-    )
-    (fp_text value LED (at -0.130901 -1.953149 208.5) (layer F.SilkS)
+    (fp_text reference D10 (at -0.075031 -1.951261 208.5) (layer F.SilkS)
+      (effects (font (size 1 1) (thickness 0.15)))
+    )
+    (fp_text value LED (at -0.099796 1.761893 208.5) (layer F.SilkS)
       (effects (font (size 1 1) (thickness 0.15)))
     )
@@
   )
   (module Soerens_Wunderschalter:Soerens_Wunderschalter (layer F.Cu)
-    (at 75.775 142.5 180)
+    (at 75.8 143.2 180)
     (fp_text reference SW2 (at 0 5 180) (layer F.SilkS) hide
       (effects (font (size 1 1) (thickness 0.15)))
     )
-    (fp_text value Schalter (at -0.1 -4.9 180) (layer F.SilkS)
+    (fp_text value Schalter (at 7.025 0.05 270) (layer F.SilkS)
       (effects (font (size 1 1) (thickness 0.15)))
     )
@@
     (pad 6 smd rect (at 4 2.5 180) (size 4 1.5) (layers F.Cu F.Paste F.Mask))
   )
-  (gr_text an (at 75.775 137.4) (layer F.SilkS)
+  (gr_text aus (at 75.8 148) (layer F.SilkS)
+    (effects (font (size 1.5 1.5) (thickness 0.15)))
+  )
+  (gr_text an (at 75.85 137.9) (layer F.SilkS)
     (effects (font (size 1.5 1.5) (thickness 0.15)))
   )
@@
   (segment (start 60.453 126.846) (end 60.453 134.618181) (width 0.5) (layer F.Cu) (net 1))
   (segment (start 60.453 134.618181) (end 61.858159 136.02334) (width 0.5) (layer F.Cu) (net 1))
+  (segment (start 83.5 141.225) (end 82.975 140.7) (width 0.5) (layer F.Cu) (net 2))
+  (segment (start 82.975 140.7) (end 79.8 140.7) (width 0.5) (layer F.Cu) (net 2))
+  (segment (start 48.675 123.4) (end 64.675 123.4) (width 0.5) (layer F.Cu) (net 2))
+  (segment (start 64.675 123.4) (end 79.8 138.525) (width 0.5) (layer F.Cu) (net 2))
+  (segment (start 79.8 138.525) (end 79.8 140.7) (width 0.5) (layer F.Cu) (net 2))
   (segment (start 48.675 123.4) (end 48.675 112.05) (width 0.5) (layer B.Cu) (net 2))
   (segment (start 48.675 112.05) (end 50.525 110.2) (width 0.5) (layer B.Cu) (net 2))
   (via (at 48.675 123.4) (size 0.6) (drill 0.4) (layers F.Cu B.Cu) (net 2))
-  (segment (start 79.775 140) (end 79.775 138.5) (width 0.5) (layer F.Cu) (net 2))
-  (segment (start 79.775 138.5) (end 64.675 123.4) (width 0.5) (layer F.Cu) (net 2))
-  (segment (start 64.675 123.4) (end 48.675 123.4) (width 0.5) (layer F.Cu) (net 2))
   (segment (start 48.675 123.4) (end 43.025 117.75) (width 0.5) (layer F.Cu) (net 2))
   (segment (start 43.025 117.75) (end 43.025 117.45) (width 0.5) (layer F.Cu) (net 2))
@@
   (segment (start 43.025 117.45) (end 43.025 113.1) (width 0.5) (layer F.Cu) (net 2))
   (segment (start 43.025 113.1) (end 42.975 113.05) (width 0.5) (layer F.Cu) (net 2))
-  (segment (start 79.775 140) (end 82.275 140) (width 0.5) (layer F.Cu) (net 2))
-  (segment (start 82.275 140) (end 83.5 141.225) (width 0.5) (layer F.Cu) (net 2))
   (segment (start 83.5 141.225) (end 83.5 151.003213) (width 0.5) (layer F.Cu) (net 2))
   (segment (start 78.703 154.386) (end 80.117213 154.386) (width 0.5) (layer F.Cu) (net 2))
@@
   (segment (start 89.695 111.925) (end 82.12 119.5) (width 0.5) (layer F.Cu) (net 13))
   (segment (start 98.93 111.925) (end 90.97 111.925) (width 0.5) (layer F.Cu) (net 13))
+  (segment (start 72.95 138.14466) (end 75.49466 138.14466) (width 0.5) (layer F.Cu) (net 15))
+  (segment (start 76.075 138.725) (end 76.075 141.975) (width 0.5) (layer F.Cu) (net 15))
+  (segment (start 75.49466 138.14466) (end 76.075 138.725) (width 0.5) (layer F.Cu) (net 15))
+  (segment (start 76.075 141.975) (end 77.3 143.2) (width 0.5) (layer F.Cu) (net 15))
+  (segment (start 77.3 143.2) (end 79.8 143.2) (width 0.5) (layer F.Cu) (net 15))
   (segment (start 63.979479 138.14466) (end 72.95 138.14466) (width 0.5) (layer F.Cu) (net 15))
   (segment (start 72.95 138.14466) (end 73.479662 138.14466) (width 0.5) (layer F.Cu) (net 15))
-  (segment (start 75.75 138.575) (end 75.31966 138.14466) (width 0.5) (layer F.Cu) (net 15))
-  (segment (start 75.31966 138.14466) (end 72.95 138.14466) (width 0.5) (layer F.Cu) (net 15))
-  (segment (start 75.75 141.975) (end 75.75 138.575) (width 0.5) (layer F.Cu) (net 15))
-  (segment (start 76.275 142.5) (end 75.75 141.975) (width 0.5) (layer F.Cu) (net 15))
-  (segment (start 79.775 142.5) (end 76.275 142.5) (width 0.5) (layer F.Cu) (net 15))
   (segment (start 73.479662 138.14466) (end 73.485002 138.15) (width 0.5) (layer F.Cu) (net 15))
 )
